File: pi-spade.sch (KiCad schematic (older format))
At the start: 2 parts, among them P1 CONN_02X20, P2 CONN_01X20

Commit message: README typo
Parts:
- P1: symbol CONN_02X20 -> pi-spade-rescue:CONN_02X20
- P2: symbol CONN_01X20 -> pi-spade-rescue:CONN_01X20
Changed lines of the file:
@@
-EESchema Schematic File Version 2
-LIBS:power
-LIBS:device
-LIBS:transistors
-LIBS:conn
-LIBS:linear
-LIBS:regul
-LIBS:74xx
-LIBS:cmos4000
-LIBS:adc-dac
-LIBS:memory
-LIBS:xilinx
-LIBS:microcontrollers
-LIBS:dsp
-LIBS:microchip
-LIBS:analog_switches
-LIBS:motorola
-LIBS:texas
-LIBS:intel
-LIBS:audio
-LIBS:interface
-LIBS:digital-audio
-LIBS:philips
-LIBS:display
-LIBS:cypress
-LIBS:siliconi
-LIBS:opto
-LIBS:atmel
-LIBS:contrib
-LIBS:valves
+EESchema Schematic File Version 4
 LIBS:pi-spade-cache
-EELAYER 25 0
+EELAYER 29 0
 EELAYER END
 $Descr A4 11693 8268
@@
 GND
 $Comp
-L CONN_02X20 P1
+L pi-spade-rescue:CONN_02X20 P1
 U 1 1 57E69125
 P 5500 3100
@@
 $EndComp
 $Comp
-L CONN_01X20 P2
+L pi-spade-rescue:CONN_01X20 P2
 U 1 1 57E6916A
 P 6700 3100
